File: boards/mainboard/mainboard.kicad_pcb (KiCad board)
At the start: 2 copper layers, 51 x 48 mm, 33 parts, among them J1 Conn_01x04_Female, J10 Conn_01x03_Female, J11 Conn_01x03_Female, J12 Conn_01x03_Female, J13 Conn_01x03_Female, J14 Conn_01x03_Female, J15 Conn_01x02_Female, J2 Conn_01x04_Female, J3 Conn_01x03_Female, J4 Conn_01x03_Female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

Commit message: address issues
Parts:
- removed J13, J14: Conn_01x03_Female, Connector_JST:JST_XH_B3B-XH-A_1x03_P2.50mm_Vertical
- removed M3∅, REF** (x3): MountingHole_3.2mm_M3, MountingHole:MountingHole_3.2mm_M3
- added H1: MountingHole, MountingHole:MountingHole_3.2mm_M3, F.Cu at (137.0, 78.5)
- added H2: MountingHole, MountingHole:MountingHole_3.2mm_M3, F.Cu at (181.0, 78.5)
- added H3: MountingHole, MountingHole:MountingHole_3.2mm_M3, F.Cu at (137.0, 119.5)
- added H4: MountingHole, MountingHole:MountingHole_3.2mm_M3, F.Cu at (181.0, 119.5)
- added R10: 1k, Resistor_SMD:R_0603_1608Metric, F.Cu at (158.9, 107.2)
- added R11: 1k, Resistor_SMD:R_0603_1608Metric, F.Cu at (158.9, 110.8)
- added R12: 1k, Resistor_SMD:R_0603_1608Metric, F.Cu at (167.8, 103.8)
- added R13: 1k, Resistor_SMD:R_0603_1608Metric, F.Cu at (167.8, 107.2)
- added R14: 1k, Resistor_SMD:R_0603_1608Metric, F.Cu at (167.8, 110.8)
- added R15: 1k, Resistor_SMD:R_0603_1608Metric, F.Cu at (174.6, 83.2)
- added R16: 1k, Resistor_SMD:R_0603_1608Metric, F.Cu at (173.6, 84.8)
- added R17: 1k, Resistor_SMD:R_0603_1608Metric, F.Cu at (174.6, 86.3)
- added R6: 1k, Resistor_SMD:R_0603_1608Metric, F.Cu at (149.9, 103.8)
- added R7: 1k, Resistor_SMD:R_0603_1608Metric, F.Cu at (149.9, 107.2)
- added R8: 1k, Resistor_SMD:R_0603_1608Metric, F.Cu at (149.9, 110.8)
- added R9: 1k, Resistor_SMD:R_0603_1608Metric, F.Cu at (158.9, 103.8)
- J10, J12, J8, J9: value Conn_01x03_Female -> Conn_01x04_Female; footprint Connector_JST:JST_XH_B3B-XH-A_1x03_P2.50mm_Vertical -> Connector_JST:JST_XH_B4B-XH-A_1x04_P2.50mm_Vertical
- moved C2 32.5 mm to (143.0, 76.0)
- moved J3 23.0 mm to (168.0, 90.0)
- moved C1 19.5 mm to (152.9, 86.3), turned to 0 degrees
- moved C3 16.4 mm to (160.9, 76.2)
- moved J5 14.0 mm to (145.0, 90.0)
- moved J6 14.0 mm to (145.0, 97.0)
- moved J4 13.5 mm to (156.5, 90.0)
- moved J8 12.8 mm to (146.0, 104.2), turned to 270 degrees
- moved J10 9.97 mm to (163.8, 104.2), turned to 270 degrees
- moved J12 8.67 mm to (172.8, 104.2), turned to 270 degrees
- moved J11 7.00 mm to (168.0, 97.0)
- moved J7 7.00 mm to (156.5, 97.0)
- moved J9 1.60 mm to (154.9, 104.2), turned to 270 degrees
- moved R1 1.13 mm to (141.8, 78.3)
- moved R4 0.60 mm to (167.8, 84.9)
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Connections:
- J10 pad 2: +3V3 -> Net-(J10-Pad2)
- J10 pad 3: /D3 -> Net-(J10-Pad3)
- J11 pad 3: /D4 -> /A5
- J12 pad 2: +3V3 -> Net-(J12-Pad2)
- J12 pad 3: /D5 -> Net-(J12-Pad3)
- J7 pad 3: /D0 -> /A4
- J8 pad 2: +3V3 -> Net-(J8-Pad2)
- J8 pad 3: /D1 -> Net-(J8-Pad3)
- J9 pad 2: +3V3 -> Net-(J9-Pad2)
- J9 pad 3: /D2 -> Net-(J9-Pad3)
- U1 pad 11: /A2 -> /A0
- U1 pad 12: /A3 -> /D0
- U1 pad 13: /D3 -> /D1
- U1 pad 15: /D1 -> /D3
- U1 pad 18: /D0 -> (no net)
- U1 pad 19: /D7 -> (no net)
- U1 pad 20: /D6 -> (no net)
- U1 pad 23: /D5 -> /D11
- U1 pad 24: /D4 -> /D10
- U1 pad 25: (no net) -> /D9
- U1 pad 27: (no net) -> /D8
- U1 pad 28: (no net) -> /D7
- U1 pad 29: (no net) -> /D6
- U1 pad 30: (no net) -> /D5
- U1 pad 31: (no net) -> /D4
- U1 pad 6: (no net) -> /A3
- U1 pad 7: (no net) -> /A4
- U1 pad 8: (no net) -> /A5
- U1 pad 9: /A0 -> /A2
Routing:
- net +3V3: track 16.1 -> 164.8 mm, vias 7 -> 4
- net /D8: track 0.00 -> 47.3 mm, vias 0 -> 2
- net /A5: track 0.00 -> 40.0 mm
- net /D9: track 0.00 -> 30.6 mm, vias 0 -> 2
- net /A4: track 0.00 -> 30.5 mm
- net Net-(J12-Pad4): track 0.00 -> 27.9 mm, vias 0 -> 1
- net Net-(J12-Pad3): track 0.00 -> 26.6 mm, vias 0 -> 1
- net Net-(J12-Pad2): track 0.00 -> 25.3 mm
- net /D11: track 0.00 -> 25.1 mm, vias 0 -> 2
- net /D10: track 0.00 -> 24.3 mm, vias 0 -> 2
- net /A0: track 7.40 -> 28.6 mm
- net /A2: track 23.3 -> 7.24 mm
- net /D4: track 25.7 -> 36.7 mm, vias 1 -> 2
- net /D3: track 35.4 -> 24.6 mm, vias 1 -> 2
- net /A3: track 30.4 -> 20.5 mm
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- added copper zone on B.Cu, net GND
- removed copper zone on B.Cu, net +3V3
Other:
- board text added: "A0"
- board text added: "A1"
- board text added: "A2"
- board text added: "A3"
- board text added: "A4"
- board text added: "A5"
- board text added: "D0"
- board text added: "D1"
- board text added: "D10"
- board text added: "D11"
- board text added: "D2"
- board text added: "D3"
- board text added: "D4"
- board text added: "D5"
- board text added: "D6"
- board text added: "D7"
- board text added: "D8"
- board text added: "D9"
- board text removed: "PA10"
- board text removed: "PA13"
- board text removed: "PA14"
- board text removed: "PA3"
- board text removed: "PA4"
- board text removed: "PA5"
- board text removed: "PA6"
- board text removed: "PA7"
- board text removed: "PA8"
- board text removed: "PA9"
- board text removed: "PB0"
- board text removed: "PB1"
