File: boards/mainboard/mainboard.sch (KiCad schematic (older format))
At the start: 29 parts, among them J1 Conn_01x04_Female, J10 Conn_01x03_Female, J11 Conn_01x03_Female, J12 Conn_01x03_Female, J13 Conn_01x03_Female, J14 Conn_01x03_Female, J15 Conn_01x02_Female, J2 Conn_01x04_Female, J3 Conn_01x03_Female, J4 Conn_01x03_Female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

Commit message: address issues
Parts:
- removed J10, J12, J13, J14, J8, J9: Conn_01x03_Female, Connector_JST:JST_XH_B3B-XH-A_1x03_P2.50mm_Vertical, symbol Connector:Conn_01x03_Female
- added H1, H2, H3, H4: MountingHole, MountingHole:MountingHole_3.2mm_M3, symbol Mechanical:MountingHole
- added J10, J12, J8, J9: Conn_01x04_Female, Connector_JST:JST_XH_B4B-XH-A_1x04_P2.50mm_Vertical, symbol Connector:Conn_01x04_Female
- added R10, R11, R12, R13, R14, R15, R16, R17, R6, R7, R8, R9: 1k, Resistor_SMD:R_0603_1608Metric, symbol Device:R_Small_US
Connections:
- net A0: now also U1.11 (PA5); no longer U1.9 (PA3)
- net A2: now also U1.9 (PA3); no longer U1.11 (PA5)
- net A3: now also U1.6 (PA0); no longer U1.12 (PA6)
- net D0: now also U1.12 (PA6), R6.1; no longer J7.3 (Pin_3), U1.18 (PA8)
- net D1: now also U1.13 (PA7), R7.1; no longer U1.15 (PB1)
- net D2: now also R8.1
- net D3: now also U1.15 (PB1), R9.1; no longer U1.13 (PA7)
- net D4: now also U1.31 (PB8), R10.1; no longer J11.3 (Pin_3), U1.24 (PA14)
- net D5: now also U1.30 (PB7), R11.1; no longer U1.23 (PA13)
- net D6: now also U1.29 (PB6), R12.1; no longer U1.20 (PA10)
- net D7: now also U1.28 (PB5), R13.1; no longer U1.19 (PA9)
- net GND: now also J10.1 (Pin_1), J12.1 (Pin_1), J8.1 (Pin_1), J9.1 (Pin_1)
- net D9: now reaches U1.25 (PA15)
- net D9: now also R15.1
- net D8: now reaches U1.27 (PB4)
- net D8: now also R14.1
- net A4: now reaches U1.7 (PA1)
- net A4: now also J7.3 (Pin_3)
- net A5: now reaches U1.8 (PA2)
- net A5: now also J11.3 (Pin_3)
- new net: J9.2 (Pin_2), R9.2
- new net: J9.3 (Pin_3), R10.2
- new net: J9.4 (Pin_4), R11.2
- new net: J8.2 (Pin_2), R6.2
- new net: J8.3 (Pin_3), R7.2
- new net: J8.4 (Pin_4), R8.2
- new net: J10.2 (Pin_2), R12.2
- new net: J10.3 (Pin_3), R13.2
- new net: J10.4 (Pin_4), R14.2
- new net: J12.2 (Pin_2), R15.2
- new net: J12.3 (Pin_3), R16.2
- new net: J12.4 (Pin_4), R17.2
- new net D10: R16.1, U1.24 (PA14)
- new net D11: R17.1, U1.23 (PA13)
